File: Hardware/MicroMod_Processor_STM32WB5MMG.sch (EAGLE design)
At the start: 0 parts

Commit message: Nearing layout completion.
Parts:
- added C1, C2: 0.1uF, SparkFun-Capacitors:0.1UF-0402T-10V-10%-X7R
- added D1: 120mA/40V/370mV, SparkFun-DiscreteSemi:DIODE-SCHOTTKY-RB751S40
- added D2: BLUE, SparkFun-LED:LED-BLUE0603
- added FD1, FD2, FD3, FD4: FIDUCIALUFIDUCIAL, SparkFun-Aesthetics:FIDUCIALUFIDUCIAL
- added FRAME2: FRAME-LETTER, SparkFun-Aesthetics:FRAME-LETTER
- added J1: MICROMOD-2222, SparkFun-MicroMod:MICROMOD-2222
- added LOGO1: FOUR_LAYER_WARNING, SparkFun-Aesthetics:FOUR_LAYER_WARNING
- added LOGO2: OSHW-LOGOMINI, SparkFun-Aesthetics:OSHW-LOGOMINI
- added LOGO3: SFE_LOGO_NAME_FLAME.1_INCH, SparkFun-Aesthetics:SFE_LOGO_NAME_FLAME.1_INCH
- added LOGO4: SPECIAL_INSTRUCTIONS-ORDERING, SparkFun-Aesthetics:SPECIAL_INSTRUCTIONS-ORDERING
- added Q1: 20V/4.2A/52mΩ/1.4W, SparkFun-DiscreteSemi:MOSFET_PCH-DMG2305UX-7
- added R1, R2: 100k, SparkFun-Resistors:100KOHM-0402T-1/16W-1%
- added R3: 2.2k, SparkFun-Resistors:2.2KOHM-0402T-1/16W-1%
- added U1: STM32WB5MMG, stm32wb5mmg:STM32WB5MMG_LOGICAL
- added U2: W25QXX128MBIT-6X5, SparkFun-IC-Memory:W25QXX128MBIT-6X5
Connections:
- new net !BOOT!: J1.!BOOT!, Q1.G, R2.1
- new net !RESET!: C1.1, J1.!RESET!, U1G3.!RST!
- new net 3.3V: C2.1, D1.A, J1.3.3V, Q1.S, R2.2, U1G3.VDD, U1G3.VDDA, U1G3.VDD_USB, U1G3.VREF+, U2.VDD
- new net A0: J1.A0, U1G2.PC2/LPTIM1_IN2
- new net A1: J1.A1, U1G2.PC3/LPTIM1_ETR
- new net AUD_BCLK: J1.AUD_BCLK, U1G1.SAI1_PDM_CK2/SAI1_SCK_A/PA8
- new net AUD_FSYNC: J1.AUD_LRCLK, U1G1.IR_OUT/SAI1_FS_A/PB9
- new net AUD_I2S_IN: J1.AUD_IN/CAM_PCLK, U1G2.PB5
- new net AUD_I2S_OUT: J1.AUD_OUT/CAM_MCLK, U1G1.SAI1_SD_A/PB15
- new net AUD_MCLK: J1.AUD_MCLK, U1G1.SAI1_PDM_CK1/SAI1_MCLK_A/PB8
- new net BATT_VIN: J1.BATT_VIN/3, U1G2.COMP1_INM/PC4
- new net BOOT0: Q1.D, R1.2, U1G3.BOOT0/PH3
- new net GND: C1.2, C2.2, D2.C, J1.GND, R1.1, U1G3.ANT_IN, U1G3.GND, U1G3.RF_OUT, U2.GND
- new net I2C1_INT: J1.I2C_!INT!, U1G2.PA1
- new net I2C1_SCL: J1.I2C_SCL, U1G1.I2C1_SCL/PB6
- new net I2C1_SDA: J1.I2C_SDA, U1G1.I2C1_SDA/PB7
- new net I2C3_SCL: J1.I2C_SCL1, U1G1.I2C3_SCL/PB13
- new net I2C3_SDA: J1.I2C_SDA1, U1G1.I2C3_SDA/PB14
- new net LPUART_RX/DEV_TX: J1.RX2, U1G1.PC0/LPUART1_RX
- new net LPUART_TX/DEV_RX: J1.TX2, U1G1.PC1/LPUART1_TX
- new net N$1: D2.A, R3.1
- new net PA0/G5: J1.G5/BUS5, U1G2.PA0
- new net PC11/G1: J1.G1/BUS1, U1G2.PC11
- new net PC13/G2: J1.G2/BUS2, U1G2.PC13
- new net PD8/G3: J1.G3/BUS3, U1G2.PD8
- new net PE3/G4: J1.G4/BUS4, U1G2.PE3
- new net PE4/G0: J1.G0/BUS0, U1G2.PE4
- new net PH0/G7: J1.G7/BUS7, U1G2.PH0
- new net PH1/G6: J1.G6/BUS6, U1G2.PH1
- new net PWM0: J1.PWM0, U1G2.PD14/TIM1_CH1
- new net PWM1: J1.PWM1, U1G2.PD15/TIM1_CH2
- new net QSPI_!CS!: U1G1.QSPI_BK1_!CS!/PD3, U2.!CS!
- new net QSPI_CLK: U1G1.QSPI_CLK/PA3, U2.CLK
- new net QSPI_IO0: U1G1.QSPI_BK1_IO0/PD4, U2.D0/DI
- new net QSPI_IO1: U1G1.QSPI_BK1_IO1/PD5, U2.D1/DO
- new net QSPI_IO2: U1G1.QSPI_BK1_IO2/PD6, U2.D2/!WP!
- new net QSPI_IO3: U1G1.QSPI_BK1_IO3/PD7, U2.D3/!HOLD!
- new net SPI_!CS!: J1.SPI_!CS!, U1G1.SPI1_!CS!/PA4
- new net SPI_PICO: J1.SPI_SDO, U1G1.SPI1_PICO/PA7
- new net SPI_POCI: J1.SPI_SDI, U1G1.SPI1_POCI/PA6
- new net SPI_SCK: J1.SPI_SCK, U1G1.SPI1_SCK/PA5
- new net STAT: R3.2, U1G2.PA2
- new net SWDCK: J1.SWDCK, U1G1.PA14/JTCK_SWCLK
- new net SWDIO: J1.SWDIO, U1G1.PA13/JTMS_SWDIO
- new net TIM1_BKIN: J1.D0, U1G2.PB12/TIM1_BKIN
- new net TIM1_ETR: J1.D1/CAM_TRIG, U1G2.PE0/TIM1_ETR
- new net UART_CTS: J1.CTS1, U1G1.PB4/USART1_CTS/!JTRST!
- new net UART_RTS_DE: J1.RTS1, U1G1.PB3/USART1_RTS_DE/JTDO_TRACE_SW0
- new net UART_RX/DEV_TX: J1.RX1, U1G1.PA10/USART1_RX
- new net UART_TX/DEV_RX: J1.TX1, U1G1.PA9/USART1_TX
- new net USB_N: J1.USB_D-, U1G1.PA11/USB_DM
- new net USB_P: J1.USB_D+, U1G1.PA12/USB_DP
- new net V_BATT: D1.C, J1.RTC_3V, U1G3.VBAT
Other:
- note added: "128 Mbit Flash"
- note added: "Boot Inversion"
- note added: "MicroMod Connector"
- note added: "Note: Decoupling capacitors are integrated onboard the module."
- note added: "STM32WB5MMG"
- note added: "Status LED"
- note added: "VDD Range: 1.8 - 3.6V"

Commit message: Layout complete.
Parts:
- added TP1, TP2, TP3, TP4, TP5, TP6, TP7, TP8: TEST-POINT3, SparkFun-Connectors:TEST-POINT3
Connections:
- net BOOT0: now also TP1.1
- net QSPI_!CS!: now also TP4.1
- net QSPI_CLK: now also TP3.1
- net QSPI_IO0: now also TP5.1
- net QSPI_IO1: now also TP6.1
- net QSPI_IO2: now also TP7.1
- net QSPI_IO3: now also TP8.1
- net STAT: now also TP2.1
Other:
- note added: "Test Points"
Changed lines of the file:
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@@
 <attribute name="REV" value="v01"/>
 </part>
+<part name="TP3" library="SparkFun-Connectors" deviceset="TEST-POINT" device="3"/>
+<part name="TP4" library="SparkFun-Connectors" deviceset="TEST-POINT" device="3"/>
+<part name="TP5" library="SparkFun-Connectors" deviceset="TEST-POINT" device="3"/>
+<part name="TP6" library="SparkFun-Connectors" deviceset="TEST-POINT" device="3"/>
+<part name="TP7" library="SparkFun-Connectors" deviceset="TEST-POINT" device="3"/>
+<part name="TP8" library="SparkFun-Connectors" deviceset="TEST-POINT" device="3"/>
+<part name="TP1" library="SparkFun-Connectors" deviceset="TEST-POINT" device="3"/>
+<part name="TP2" library="SparkFun-Connectors" deviceset="TEST-POINT" device="3"/>
 </parts>
 <sheets>
@@
 <plain>
 <text x="5.08" y="2.54" size="1.778" layer="97" font="vector">Note: Decoupling capacitors are integrated onboard the module.</text>
-<wire x1="147.32" y1="35.56" x2="147.32" y2="63.5" width="0.2032" layer="97" style="longdash"/>
 <wire x1="147.32" y1="63.5" x2="248.92" y2="63.5" width="0.2032" layer="97" style="longdash"/>
 <wire x1="88.9" y1="0" x2="88.9" y2="63.5" width="0.2032" layer="97" style="longdash"/>
 <wire x1="88.9" y1="63.5" x2="88.9" y2="101.6" width="0.2032" layer="97" style="longdash"/>
-<wire x1="88.9" y1="101.6" x2="124.46" y2="101.6" width="0.2032" layer="97" style="longdash"/>
-<wire x1="124.46" y1="101.6" x2="124.46" y2="185.42" width="0.2032" layer="97" style="longdash"/>
+<wire x1="88.9" y1="101.6" x2="119.38" y2="101.6" width="0.2032" layer="97" style="longdash"/>
+<wire x1="119.38" y1="101.6" x2="119.38" y2="137.16" width="0.2032" layer="97" style="longdash"/>
+<wire x1="119.38" y1="137.16" x2="119.38" y2="185.42" width="0.2032" layer="97" style="longdash"/>
 <wire x1="147.32" y1="63.5" x2="88.9" y2="63.5" width="0.2032" layer="97" style="longdash"/>
-<wire x1="124.46" y1="101.6" x2="147.32" y2="101.6" width="0.2032" layer="97" style="longdash"/>
+<wire x1="119.38" y1="101.6" x2="147.32" y2="101.6" width="0.2032" layer="97" style="longdash"/>
 <wire x1="147.32" y1="101.6" x2="147.32" y2="63.5" width="0.2032" layer="97" style="longdash"/>
 <text x="63.5" y="172.72" size="1.778" layer="97" font="vector" align="bottom-center">VDD Range: 1.8 - 3.6V</text>
@@
 LED</text>
 <wire x1="127" y1="0" x2="127" y2="63.5" width="0.2032" layer="97" style="longdash"/>
+<wire x1="147.32" y1="35.56" x2="147.32" y2="63.5" width="0.2032" layer="97" style="longdash"/>
+<wire x1="147.32" y1="101.6" x2="147.32" y2="137.16" width="0.2032" layer="97" style="longdash"/>
+<wire x1="147.32" y1="137.16" x2="119.38" y2="137.16" width="0.2032" layer="97" style="longdash"/>
+<text x="132.08" y="129.54" size="2.54" layer="94" font="vector" align="bottom-center">Test Points</text>
 </plain>
 <instances>
@@
 <attribute name="REV" x="236.22" y="6.604" size="2.7432" layer="94" font="vector"/>
 </instance>
+<instance part="TP3" gate="G$1" x="134.62" y="119.38" smashed="yes">
+<attribute name="NAME" x="139.7" y="119.38" size="1.778" layer="95" font="vector" align="center-left"/>
+</instance>
+<instance part="TP4" gate="G$1" x="134.62" y="116.84" smashed="yes">
+<attribute name="NAME" x="139.7" y="116.84" size="1.778" layer="95" font="vector" align="center-left"/>
+</instance>
+<instance part="TP5" gate="G$1" x="134.62" y="114.3" smashed="yes">
+<attribute name="NAME" x="139.7" y="114.3" size="1.778" layer="95" font="vector" align="center-left"/>
+</instance>
+<instance part="TP6" gate="G$1" x="134.62" y="111.76" smashed="yes">
+<attribute name="NAME" x="139.7" y="111.76" size="1.778" layer="95" font="vector" align="center-left"/>
+</instance>
+<instance part="TP7" gate="G$1" x="134.62" y="109.22" smashed="yes">
+<attribute name="NAME" x="139.7" y="109.22" size="1.778" layer="95" font="vector" align="center-left"/>
+</instance>
+<instance part="TP8" gate="G$1" x="134.62" y="106.68" smashed="yes">
+<attribute name="NAME" x="139.7" y="106.68" size="1.778" layer="95" font="vector" align="center-left"/>
+</instance>
+<instance part="TP1" gate="G$1" x="134.62" y="124.46" smashed="yes">
+<attribute name="NAME" x="139.7" y="124.46" size="1.778" layer="95" font="vector" align="center-left"/>
+</instance>
+<instance part="TP2" gate="G$1" x="134.62" y="121.92" smashed="yes">
+<attribute name="NAME" x="139.7" y="121.92" size="1.778" layer="95" font="vector" align="center-left"/>
+</instance>
 </instances>
 <busses>
@@
 <segment>
 <pinref part="U1" gate="G3" pin="BOOT0/PH3"/>
+<pinref part="Q1" gate="G$1" pin="D"/>
 <wire x1="53.34" y1="25.4" x2="99.06" y2="25.4" width="0.1524" layer="91"/>
-<pinref part="Q1" gate="G$1" pin="D"/>
 <wire x1="99.06" y1="27.94" x2="99.06" y2="25.4" width="0.1524" layer="91"/>
 <wire x1="99.06" y1="25.4" x2="99.06" y2="22.86" width="0.1524" layer="91"/>
 <junction x="99.06" y="25.4"/>
 <pinref part="R1" gate="G$1" pin="2"/>
+<label x="99.06" y="25.4" size="1.27" layer="95" xref="yes"/>
+</segment>
+<segment>
+<pinref part="TP1" gate="G$1" pin="1"/>
+<wire x1="132.08" y1="124.46" x2="134.62" y2="124.46" width="0.1524" layer="91" style="longdash"/>
+<label x="132.08" y="124.46" size="1.27" layer="95" rot="R180" xref="yes"/>
 </segment>
 </net>
@@
 <pinref part="U2" gate="U1" pin="CLK"/>
 </segment>
+<segment>
+<pinref part="TP3" gate="G$1" pin="1"/>
+<wire x1="132.08" y1="119.38" x2="134.62" y2="119.38" width="0.1524" layer="91" style="longdash"/>
+<label x="132.08" y="119.38" size="1.27" layer="95" rot="R180" xref="yes"/>
+</segment>
 </net>
 <net name="QSPI_!CS!" class="0">
@@
 <pinref part="U2" gate="U1" pin="!CS!"/>
 </segment>
+<segment>
+<pinref part="TP4" gate="G$1" pin="1"/>
+<wire x1="132.08" y1="116.84" x2="134.62" y2="116.84" width="0.1524" layer="91" style="longdash"/>
+<label x="132.08" y="116.84" size="1.27" layer="95" rot="R180" xref="yes"/>
+</segment>
 </net>
 <net name="QSPI_IO0" class="0">
@@
 <pinref part="U2" gate="U1" pin="D0/DI"/>
 </segment>
+<segment>
+<pinref part="TP5" gate="G$1" pin="1"/>
+<wire x1="132.08" y1="114.3" x2="134.62" y2="114.3" width="0.1524" layer="91" style="longdash"/>
+<label x="132.08" y="114.3" size="1.27" layer="95" rot="R180" xref="yes"/>
+</segment>
 </net>
 <net name="QSPI_IO1" class="0">
@@
 <pinref part="U2" gate="U1" pin="D1/DO"/>
 </segment>
+<segment>
+<pinref part="TP6" gate="G$1" pin="1"/>
+<wire x1="132.08" y1="111.76" x2="134.62" y2="111.76" width="0.1524" layer="91" style="longdash"/>
+<label x="132.08" y="111.76" size="1.27" layer="95" rot="R180" xref="yes"/>
+</segment>
 </net>
 <net name="QSPI_IO2" class="0">
@@
 <pinref part="U2" gate="U1" pin="D2/!WP!"/>
 </segment>
+<segment>
+<pinref part="TP7" gate="G$1" pin="1"/>
+<wire x1="132.08" y1="109.22" x2="134.62" y2="109.22" width="0.1524" layer="91" style="longdash"/>
+<label x="132.08" y="109.22" size="1.27" layer="95" rot="R180" xref="yes"/>
+</segment>
 </net>
 <net name="QSPI_IO3" class="0">
@@
 <pinref part="U2" gate="U1" pin="D3/!HOLD!"/>
 </segment>
+<segment>
+<pinref part="TP8" gate="G$1" pin="1"/>
+<wire x1="132.08" y1="106.68" x2="134.62" y2="106.68" width="0.1524" layer="91" style="longdash"/>
+<label x="132.08" y="106.68" size="1.27" layer="95" rot="R180" xref="yes"/>
+</segment>
 </net>
 <net name="AUD_MCLK" class="0">
@@
 <segment>
 <pinref part="R3" gate="G$1" pin="2"/>
-<wire x1="137.16" y1="33.02" x2="137.16" y2="35.56" width="0.1524" layer="91"/>
-<label x="137.16" y="35.56" size="1.27" layer="95" font="vector" rot="R90" xref="yes"/>
-</segment>
-</net>
+<label x="137.16" y="38.1" size="1.27" layer="95" font="vector" rot="R90" xref="yes"/>
+<wire x1="137.16" y1="33.02" x2="137.16" y2="38.1" width="0.1524" layer="91"/>
+</segment>
+<segment>
+<pinref part="TP2" gate="G$1" pin="1"/>
+<wire x1="132.08" y1="121.92" x2="134.62" y2="121.92" width="0.1524" layer="91" style="longdash"/>
+<label x="132.08" y="121.92" size="1.27" layer="95" rot="R180" xref="yes"/>
+</segment>
+</net>

Commit message: Updates from Design Review v01
Fix footprint.
Reposition bottom silk
Removed extraneous vias.
Renamed some nets to match micromod connector.
Rerouted some traces.
Added ground vias near fast switching vias.
Moved traces to expand ground plane.
Removed all but BOOT0 test point with Chris' approval.
Parts:
- removed TP2, TP3, TP4, TP5, TP6, TP7, TP8: TEST-POINT3, SparkFun-Connectors:TEST-POINT3
Connections:
- net I2C3_SCL renamed I2C3_SCL1
- net I2C3_SDA renamed I2C3_SDA1
- net LPUART_RX/DEV_TX renamed LP_RX2/DEV_TX2
- net LPUART_TX/DEV_RX renamed LP_TX2/DEV_RX2
- net UART_RX/DEV_TX renamed RX1/DEV_TX1
- net UART_TX/DEV_RX renamed TX1/DEV_RX1
- net QSPI_!CS!: no longer TP4.1
- net QSPI_CLK: no longer TP3.1
- net QSPI_IO0: no longer TP5.1
- net QSPI_IO1: no longer TP6.1
- net QSPI_IO2: no longer TP7.1
- net QSPI_IO3: no longer TP8.1
- net STAT: no longer TP2.1
Other:
- note removed: "Test Points"
- moved on the sheet: TP1
Changed lines of the file:
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@@
 <attribute name="REV" value="v01"/>
 </part>
-<part name="TP3" library="SparkFun-Connectors" deviceset="TEST-POINT" device="3"/>
-<part name="TP4" library="SparkFun-Connectors" deviceset="TEST-POINT" device="3"/>
-<part name="TP5" library="SparkFun-Connectors" deviceset="TEST-POINT" device="3"/>
-<part name="TP6" library="SparkFun-Connectors" deviceset="TEST-POINT" device="3"/>
-<part name="TP7" library="SparkFun-Connectors" deviceset="TEST-POINT" device="3"/>
-<part name="TP8" library="SparkFun-Connectors" deviceset="TEST-POINT" device="3"/>
 <part name="TP1" library="SparkFun-Connectors" deviceset="TEST-POINT" device="3"/>
-<part name="TP2" library="SparkFun-Connectors" deviceset="TEST-POINT" device="3"/>
 </parts>
 <sheets>
@@
 <wire x1="88.9" y1="63.5" x2="88.9" y2="101.6" width="0.2032" layer="97" style="longdash"/>
 <wire x1="88.9" y1="101.6" x2="119.38" y2="101.6" width="0.2032" layer="97" style="longdash"/>
-<wire x1="119.38" y1="101.6" x2="119.38" y2="137.16" width="0.2032" layer="97" style="longdash"/>
-<wire x1="119.38" y1="137.16" x2="119.38" y2="185.42" width="0.2032" layer="97" style="longdash"/>
+<wire x1="119.38" y1="101.6" x2="119.38" y2="185.42" width="0.2032" layer="97" style="longdash"/>
 <wire x1="147.32" y1="63.5" x2="88.9" y2="63.5" width="0.2032" layer="97" style="longdash"/>
 <wire x1="119.38" y1="101.6" x2="147.32" y2="101.6" width="0.2032" layer="97" style="longdash"/>
@@
 <wire x1="127" y1="0" x2="127" y2="63.5" width="0.2032" layer="97" style="longdash"/>
 <wire x1="147.32" y1="35.56" x2="147.32" y2="63.5" width="0.2032" layer="97" style="longdash"/>
-<wire x1="147.32" y1="101.6" x2="147.32" y2="137.16" width="0.2032" layer="97" style="longdash"/>
-<wire x1="147.32" y1="137.16" x2="119.38" y2="137.16" width="0.2032" layer="97" style="longdash"/>
-<text x="132.08" y="129.54" size="2.54" layer="94" font="vector" align="bottom-center">Test Points</text>
 </plain>
 <instances>
@@
 <attribute name="REV" x="236.22" y="6.604" size="2.7432" layer="94" font="vector"/>
 </instance>
-<instance part="TP3" gate="G$1" x="134.62" y="119.38" smashed="yes">
-<attribute name="NAME" x="139.7" y="119.38" size="1.778" layer="95" font="vector" align="center-left"/>
-</instance>
-<instance part="TP4" gate="G$1" x="134.62" y="116.84" smashed="yes">
-<attribute name="NAME" x="139.7" y="116.84" size="1.778" layer="95" font="vector" align="center-left"/>
-</instance>
-<instance part="TP5" gate="G$1" x="134.62" y="114.3" smashed="yes">
-<attribute name="NAME" x="139.7" y="114.3" size="1.778" layer="95" font="vector" align="center-left"/>
-</instance>
-<instance part="TP6" gate="G$1" x="134.62" y="111.76" smashed="yes">
-<attribute name="NAME" x="139.7" y="111.76" size="1.778" layer="95" font="vector" align="center-left"/>
-</instance>
-<instance part="TP7" gate="G$1" x="134.62" y="109.22" smashed="yes">
-<attribute name="NAME" x="139.7" y="109.22" size="1.778" layer="95" font="vector" align="center-left"/>
-</instance>
-<instance part="TP8" gate="G$1" x="134.62" y="106.68" smashed="yes">
-<attribute name="NAME" x="139.7" y="106.68" size="1.778" layer="95" font="vector" align="center-left"/>
-</instance>
-<instance part="TP1" gate="G$1" x="134.62" y="124.46" smashed="yes">
-<attribute name="NAME" x="139.7" y="124.46" size="1.778" layer="95" font="vector" align="center-left"/>
-</instance>
-<instance part="TP2" gate="G$1" x="134.62" y="121.92" smashed="yes">
-<attribute name="NAME" x="139.7" y="121.92" size="1.778" layer="95" font="vector" align="center-left"/>
+<instance part="TP1" gate="G$1" x="63.5" y="30.48" smashed="yes" rot="R90">
+<attribute name="NAME" x="66.04" y="33.02" size="1.778" layer="95" font="vector" align="center-left"/>
 </instance>
 </instances>
@@
 <pinref part="U1" gate="G3" pin="BOOT0/PH3"/>
 <pinref part="Q1" gate="G$1" pin="D"/>
-<wire x1="53.34" y1="25.4" x2="99.06" y2="25.4" width="0.1524" layer="91"/>
+<wire x1="53.34" y1="25.4" x2="63.5" y2="25.4" width="0.1524" layer="91"/>
+<wire x1="63.5" y1="25.4" x2="99.06" y2="25.4" width="0.1524" layer="91"/>
 <wire x1="99.06" y1="27.94" x2="99.06" y2="25.4" width="0.1524" layer="91"/>
 <wire x1="99.06" y1="25.4" x2="99.06" y2="22.86" width="0.1524" layer="91"/>
 <junction x="99.06" y="25.4"/>
 <pinref part="R1" gate="G$1" pin="2"/>
-<label x="99.06" y="25.4" size="1.27" layer="95" xref="yes"/>
-</segment>
-<segment>
+<label x="66.04" y="27.94" size="1.27" layer="95" xref="yes"/>
 <pinref part="TP1" gate="G$1" pin="1"/>
-<wire x1="132.08" y1="124.46" x2="134.62" y2="124.46" width="0.1524" layer="91" style="longdash"/>
-<label x="132.08" y="124.46" size="1.27" layer="95" rot="R180" xref="yes"/>
+<wire x1="63.5" y1="30.48" x2="63.5" y2="27.94" width="0.1524" layer="91"/>
+<junction x="63.5" y="25.4"/>
+<wire x1="63.5" y1="27.94" x2="63.5" y2="25.4" width="0.1524" layer="91"/>
+<wire x1="66.04" y1="27.94" x2="63.5" y2="27.94" width="0.1524" layer="91"/>
+<junction x="63.5" y="27.94"/>
 </segment>
 </net>
@@
 </segment>
 </net>
-<net name="I2C3_SCL" class="0">
+<net name="I2C3_SCL1" class="0">
 <segment>
 <pinref part="U1" gate="G1" pin="I2C3_SCL/PB13"/>
@@
 </segment>
 </net>
-<net name="I2C3_SDA" class="0">
+<net name="I2C3_SDA1" class="0">
 <segment>
 <pinref part="U1" gate="G1" pin="I2C3_SDA/PB14"/>
@@
 <pinref part="U2" gate="U1" pin="CLK"/>
 </segment>
-<segment>
-<pinref part="TP3" gate="G$1" pin="1"/>
-<wire x1="132.08" y1="119.38" x2="134.62" y2="119.38" width="0.1524" layer="91" style="longdash"/>
-<label x="132.08" y="119.38" size="1.27" layer="95" rot="R180" xref="yes"/>
-</segment>
 </net>
 <net name="QSPI_!CS!" class="0">
@@
 <pinref part="U2" gate="U1" pin="!CS!"/>
 </segment>
-<segment>
-<pinref part="TP4" gate="G$1" pin="1"/>
-<wire x1="132.08" y1="116.84" x2="134.62" y2="116.84" width="0.1524" layer="91" style="longdash"/>
-<label x="132.08" y="116.84" size="1.27" layer="95" rot="R180" xref="yes"/>
-</segment>
 </net>
 <net name="QSPI_IO0" class="0">
@@
 <pinref part="U2" gate="U1" pin="D0/DI"/>
 </segment>
-<segment>
-<pinref part="TP5" gate="G$1" pin="1"/>
-<wire x1="132.08" y1="114.3" x2="134.62" y2="114.3" width="0.1524" layer="91" style="longdash"/>
-<label x="132.08" y="114.3" size="1.27" layer="95" rot="R180" xref="yes"/>
-</segment>
 </net>
 <net name="QSPI_IO1" class="0">
@@
 <pinref part="U2" gate="U1" pin="D1/DO"/>
 </segment>
-<segment>
-<pinref part="TP6" gate="G$1" pin="1"/>
-<wire x1="132.08" y1="111.76" x2="134.62" y2="111.76" width="0.1524" layer="91" style="longdash"/>
-<label x="132.08" y="111.76" size="1.27" layer="95" rot="R180" xref="yes"/>
-</segment>
 </net>
 <net name="QSPI_IO2" class="0">
@@
 <pinref part="U2" gate="U1" pin="D2/!WP!"/>
 </segment>
-<segment>
-<pinref part="TP7" gate="G$1" pin="1"/>
-<wire x1="132.08" y1="109.22" x2="134.62" y2="109.22" width="0.1524" layer="91" style="longdash"/>
-<label x="132.08" y="109.22" size="1.27" layer="95" rot="R180" xref="yes"/>
-</segment>
 </net>
 <net name="QSPI_IO3" class="0">
@@
 <pinref part="U2" gate="U1" pin="D3/!HOLD!"/>
 </segment>
-<segment>
-<pinref part="TP8" gate="G$1" pin="1"/>
-<wire x1="132.08" y1="106.68" x2="134.62" y2="106.68" width="0.1524" layer="91" style="longdash"/>
-<label x="132.08" y="106.68" size="1.27" layer="95" rot="R180" xref="yes"/>
-</segment>
 </net>
 <net name="AUD_MCLK" class="0">
@@
 </segment>
 </net>
-<net name="LPUART_RX/DEV_TX" class="0">
+<net name="LP_RX2/DEV_TX2" class="0">
 <segment>
 <wire x1="25.4" y1="157.48" x2="22.86" y2="157.48" width="0.1524" layer="91"/>
@@
 </segment>
 </net>
-<net name="LPUART_TX/DEV_RX" class="0">
+<net name="LP_TX2/DEV_RX2" class="0">
 <segment>
 <wire x1="25.4" y1="154.94" x2="22.86" y2="154.94" width="0.1524" layer="91"/>
@@
 </segment>
 </net>
-<net name="UART_TX/DEV_RX" class="0">
+<net name="TX1/DEV_RX1" class="0">
 <segment>
 <wire x1="25.4" y1="149.86" x2="22.86" y2="149.86" width="0.1524" layer="91"/>
@@
 </segment>
 </net>
-<net name="UART_RX/DEV_TX" class="0">
+<net name="RX1/DEV_TX1" class="0">
 <segment>
 <wire x1="25.4" y1="147.32" x2="22.86" y2="147.32" width="0.1524" layer="91"/>
@@
 <wire x1="137.16" y1="33.02" x2="137.16" y2="38.1" width="0.1524" layer="91"/>
 </segment>
-<segment>
-<pinref part="TP2" gate="G$1" pin="1"/>
-<wire x1="132.08" y1="121.92" x2="134.62" y2="121.92" width="0.1524" layer="91" style="longdash"/>
-<label x="132.08" y="121.92" size="1.27" layer="95" rot="R180" xref="yes"/>
-</segment>
 </net>
 <net name="PA0/G5" class="0">
@@
 <segment>
 <pinref part="U1" gate="G2" pin="COMP1_INM/PC4"/>
-<wire x1="76.2" y1="55.88" x2="73.66" y2="55.88" width="0.1524" layer="91" style="longdash"/>
+<wire x1="76.2" y1="55.88" x2="73.66" y2="55.88" width="0.1524" layer="91"/>
 <label x="76.2" y="55.88" size="1.27" layer="95" font="vector" xref="yes"/>
 </segment>

Commit message: Update for v10
Changelog from v01:
* Connect unused GPIO to ground
** AN4899
** Reduces power consumption and noise
* Add ESD to USB data lines
** This module is sensitive to it
** Moved Flash chip up to make room for ESD diode package
* Set text objects to spin
** When panelizing, the upside down ones didn’t spin on protos so I fixed that
Parts:
- added U3: ESD Diode, SparkFun-DiscreteSemi:TVS_DIODE_ARRAY_DT1042-04SO-7
- FRAME2: REV v01 -> v10
Connections:
- new net N$2: J1.USB_VIN, U3.VCC
- net GND: now also U1G1.PA15/JTDI, U1G1.PC10/TRACE_D1, U1G1.PC12/TRACE_D3, U1G1.PD10/TRIG_INOUT, U1G1.PD2/TRACE_D2/TSC_SYNC, U1G1.PD9/TRACE_D0, U1G1.PE2/TRACE_CK, U1G2.COMP1_INP/PB2, U1G2.COMP1_OUT/PB0, U1G2.LPTIM2_ETR/PD11, U1G2.LPTIM2_IN1/PD12, U1G2.LPTIM2_OUT/PD13, U1G2.PB1, U1G2.PB10, U1G2.PB11, U1G2.PC5, U1G2.PC6/TSC_G4_IO1, U1G2.PC7/TSC_G4_IO2, U1G2.PC8/TSC_G4_IO3, U1G2.PC9/TSC_G4_IO4/USB_!OE!, U1G2.PD0, U1G2.PD1, U1G2.PE1, U3.VSS
- net USB_N: now also U3.IO4
- net USB_P: now also U3.IO1
